File: board/iCEGenius.kicad_pcb (KiCad board)
At the start: 6 copper layers, 21.8 x 44.6 mm, 57 parts, among them IC1 MIC5528-3.3YMT-T5, IC2 MCP2210-I_MQ, J1 USB4105-GF-A-060, J2 LEFT, J3 RIGHT, Q1 MMBT3904-TP, U1 MIC5365-1.2YC5, U2 W25Q80DVSNIG, U3 ICE40LP384-SG32, Y1 815-ABM8AIG-12MHZ1ZT, Y2 ASFL1-100.000MHZ-L-T

Commit message: linux push
Parts:
- removed the C3 at (161.8, 87.7)
- removed the C4 at (159.6, 89.7)
- removed the C5 at (159.6, 88.5)
- removed the C6 at (159.6, 87.3)
- removed the IC1 at (161.5, 89.5)
- added U1: BU33SD5WG-TR, SamacSys_Parts:SOT95P280X125-5N, F.Cu at (160.6, 88.4)
- moved REF** 6.50 mm to (155.9, 112.6)
- moved C2 4.76 mm to (161.1, 91.1), turned to 180 degrees
- moved C11 3.36 mm to (161.5, 117.5), turned to 135 degrees
- moved C1 0.46 mm to (162.0, 85.6)
- renumbered C14 to C10, C15 to C11, C16 to C12, C17 to C13, C18 to C14, C19 to C15, C20 to C16, C21 to C17, C22 to C18, C23 to C19, C24 to C20, C25 to C21, C26 to C22, C27 to C23, C28 to C24, C29 to C25, C7 to C3, C8 to C4, C9 to C5, C10 to C6, C11 to C7, C12 to C8, C13 to C9, IC2 to IC1, U1 to U2, U2 to U3, U3 to U4
Connections:
- C2 pad 1: +5V -> +3V3
Routing:
- net +3V3: track 46.5 -> 49.1 mm, vias 11 -> 10
- net GND: track 60.8 -> 58.3 mm, vias 44 -> 43
- net +1V2: track 4.84 -> 6.63 mm
- net +5V: track 41.8 -> 42.3 mm
Other:
- board text added: "v3"
- board text removed: "v2"

Commit message: uploaded current state - unfinished
Connections:
- IC1 pad 10: SDI -> MISO
- IC1 pad 6: SDO -> MOSI
- U3 pad 2: SDO -> MISO
- U3 pad 5: SDI -> MOSI
- U4 pad 12: SDO -> MISO
- U4 pad 13: SDI -> MOSI
Routing:
- net SDI: track 23.3 -> 0.00 mm, vias 3 -> 0
- net MOSI: track 0.00 -> 21.2 mm, vias 0 -> 2
- net MISO: track 0.00 -> 20.8 mm, vias 0 -> 3
- net SDO: track 17.6 -> 0.00 mm, vias 3 -> 0
- net SCK: track 23.9 -> 24.9 mm
- net +3V3: track 49.1 -> 48.3 mm
- net GND: track 58.3 -> 57.8 mm, vias 43 -> 42
Other:
- board text added: "v4"
- board text removed: "v3"
