File: board/iCEGenius.kicad_sch (KiCad schematic)
At the start: 56 parts, among them IC1 MIC5528-3.3YMT-T5, IC2 MCP2210-I_MQ, J1 USB4105-GF-A-060, J2 LEFT, J3 RIGHT, Q1 MMBT3904-TP, U1 MIC5365-1.2YC5, U2 W25Q80DVSNIG, U3 ICE40LP384-SG32, Y1 815-ABM8AIG-12MHZ1ZT, Y2 ASFL1-100.000MHZ-L-T

Commit message: vscode extension progress
Other:
- note added: "USB-SPI Bridge"
- note removed: "USB-SPI Controller"
Changed lines of the file:
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@@
   (title_block
     (title "Overview")
+    (rev "2")
   )
   (junction (at 34.29 77.47) (diameter 0) (color 0 0 0 0)
@@
     (fill (type none))
   )
-  (text "USB-SPI Controller" (at 86.36 107.95 0)
+  (text "USB-SPI Bridge" (at 86.36 107.95 0)
     (effects (font (size 1.27 1.27) (thickness 0.254) bold) (justify left bottom))
   )

Commit message: linux push
Parts:
- removed C2, C3, C5, C6: 1u, Capacitor_SMD:C_0402_1005Metric, symbol Device:C_Small
- removed IC1: MIC5528-3.3YMT-T5, SamacSys_Parts:SON40P120X120X60-7N-D, symbol SamacSys_Parts:MIC5528-3.3YMT-T5
- added U1: BU33SD5WG-TR, SOT95P280X125-5N, symbol SamacSys_Parts:BU33SD5WG-TR
- renumbered C14 to C10, C15 to C11, C16 to C12, C17 to C13, C18 to C14, C19 to C15, C20 to C16, C21 to C17, C22 to C18, C23 to C19, C4 to C2, C24 to C20, C25 to C21, C26 to C22, C27 to C23, C28 to C24, C29 to C25, C7 to C3, C8 to C4, C9 to C5, C10 to C6, C11 to C7, C12 to C8, C13 to C9, IC2 to IC1, U1 to U2, U2 to U3, U3 to U4
Connections:
- net +3V3: now also U1.5 (VOUT)
- net +5V: now also U1.1 (VIN), U1.3 (STBY)
- net GND: now also U1.2 (GND)
Other:
- moved on the sheet: C1, C2

Commit message: uploaded current state - unfinished
Connections:
- net SDI renamed MOSI
- net MOSI: now also IC1.6 (MOSI); no longer IC1.10 (MISO)
- net SDO renamed MISO
- net MISO: now also IC1.10 (MISO); no longer IC1.6 (MOSI)
Changed lines of the file:
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@@
+    )
+  )
+  (global_label "MISO" (shape input) (at 43.18 97.79 180) (fields_autoplaced)
+    (effects (font (size 1.27 1.27)) (justify right))
+    (property "Intersheetrefs" "${INTERSHEET_REFS}" (at 36.2533 97.79 0)
+      (effects (font (size 1.27 1.27)) (justify right) hide)
     )
   )
@@
     )
   )
-  (global_label "SDI" (shape input) (at 43.18 95.25 180) (fields_autoplaced)
-    (effects (font (size 1.27 1.27)) (justify right))
-    (property "Intersheetrefs" "${INTERSHEET_REFS}" (at 37.1899 95.25 0)
-      (effects (font (size 1.27 1.27)) (justify right) hide)
-    )
-  )
   (global_label "SCK" (shape bidirectional) (at 115.57 85.09 180) (fields_autoplaced)
     (effects (font (size 1.27 1.27)) (justify right))
@@
     )
   )
+  (global_label "MOSI" (shape output) (at 152.4 151.13 180) (fields_autoplaced)
+    (effects (font (size 1.27 1.27)) (justify right))
+    (property "Intersheetrefs" "${INTERSHEET_REFS}" (at 145.4733 151.13 0)
+      (effects (font (size 1.27 1.27)) (justify right) hide)
+    )
+  )
   (global_label "SS" (shape bidirectional) (at 152.4 158.75 180) (fields_autoplaced)
     (effects (font (size 1.27 1.27)) (justify right))
@@
     )
   )
-  (global_label "SDI" (shape input) (at 152.4 151.13 180) (fields_autoplaced)
-    (effects (font (size 1.27 1.27)) (justify right))
-    (property "Intersheetrefs" "${INTERSHEET_REFS}" (at 146.4099 151.13 0)
-      (effects (font (size 1.27 1.27)) (justify right) hide)
-    )
-  )
   (global_label "IOR_35_GBIN3" (shape bidirectional) (at 226.06 74.93 180) (fields_autoplaced)
     (effects (font (size 1.27 1.27)) (justify right))
@@
     )
   )
-  (global_label "SDO" (shape output) (at 152.4 153.67 180) (fields_autoplaced)
-    (effects (font (size 1.27 1.27)) (justify right))
-    (property "Intersheetrefs" "${INTERSHEET_REFS}" (at 145.6842 153.67 0)
-      (effects (font (size 1.27 1.27)) (justify right) hide)
-    )
-  )
   (global_label "IOL_2B" (shape bidirectional) (at 255.27 67.31 0) (fields_autoplaced)
     (effects (font (size 1.27 1.27)) (justify left))
@@
     )
   )
-  (global_label "SDO" (shape output) (at 115.57 90.17 180) (fields_autoplaced)
-    (effects (font (size 1.27 1.27)) (justify right))
-    (property "Intersheetrefs" "${INTERSHEET_REFS}" (at 108.8542 90.17 0)
+  (global_label "MOSI" (shape output) (at 115.57 90.17 180) (fields_autoplaced)
+    (effects (font (size 1.27 1.27)) (justify right))
+    (property "Intersheetrefs" "${INTERSHEET_REFS}" (at 108.6433 90.17 0)
       (effects (font (size 1.27 1.27)) (justify right) hide)
     )
@@
     )
   )
-  (global_label "SDI" (shape input) (at 115.57 87.63 180) (fields_autoplaced)
-    (effects (font (size 1.27 1.27)) (justify right))
-    (property "Intersheetrefs" "${INTERSHEET_REFS}" (at 109.5799 87.63 0)
+  (global_label "MISO" (shape input) (at 115.57 87.63 180) (fields_autoplaced)
+    (effects (font (size 1.27 1.27)) (justify right))
+    (property "Intersheetrefs" "${INTERSHEET_REFS}" (at 108.6433 87.63 0)
       (effects (font (size 1.27 1.27)) (justify right) hide)
     )
@@
     )
   )
+  (global_label "MISO" (shape input) (at 152.4 153.67 180) (fields_autoplaced)
+    (effects (font (size 1.27 1.27)) (justify right))
+    (property "Intersheetrefs" "${INTERSHEET_REFS}" (at 145.4733 153.67 0)
+      (effects (font (size 1.27 1.27)) (justify right) hide)
+    )
+  )
   (global_label "IOR_34" (shape bidirectional) (at 209.55 138.43 0) (fields_autoplaced)
     (effects (font (size 1.27 1.27)) (justify left))
@@
     )
   )
+  (global_label "MOSI" (shape output) (at 43.18 95.25 180) (fields_autoplaced)
+    (effects (font (size 1.27 1.27)) (justify right))
+    (property "Intersheetrefs" "${INTERSHEET_REFS}" (at 36.2533 95.25 0)
+      (effects (font (size 1.27 1.27)) (justify right) hide)
+    )
+  )
   (global_label "IOT_50_GBIN1" (shape bidirectional) (at 255.27 74.93 0) (fields_autoplaced)
     (effects (font (size 1.27 1.27)) (justify left))
@@
       (effects (font (size 1.27 1.27)) (justify right) hide)
     )
-  )
-  (global_label "SDO" (shape output) (at 43.18 97.79 180) (fields_autoplaced)
-    (effects (font (size 1.27 1.27)) (justify right))
-    (property "Intersheetrefs" "${INTERSHEET_REFS}" (at 36.4642 97.79 0)
-      (effects (font (size 1.27 1.27)) (justify right) hide)
-    )
